File: Reciever.kicad_sch (KiCad schematic)
At the start: 15 parts

Commit message: Added PCB v1
Parts:
- added C9: C, Capacitor_THT:C_Radial_D8.0mm_H11.5mm_P3.50mm, symbol Device:C
- C4, C5, C6, C7, C8: footprint (none) -> Capacitor_THT:C_Radial_D8.0mm_H11.5mm_P3.50mm
- R10, R11, R6, R7, R8, R9: footprint (none) -> Resistor_THT:R_Axial_DIN0309_L9.0mm_D3.2mm_P12.70mm_Horizontal
- RecieveCoil1: renamed from RecieveCoil; footprint (none) -> Connector_PinSocket_2.54mm:PinSocket_1x02_P2.54mm_Vertical
- U2: footprint Package_DIP:DIP-8_W7.62mm_Socket_LongPads -> Package_SO:SOIC-8-1EP_3.9x4.9mm_P1.27mm_EP2.29x3mm
- renumbered AudioOut to AudioOut1, PowerIn to PowerIn1
Connections:
- net GND2: now also C9.2
- net VDD: now also C9.1
Changed lines of the file:
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@@
+	)
+	(junction
+		(at 45.72 39.37)
+		(diameter 0)
+		(color 0 0 0 0)
 	)
 	(junction
@@
 	)
 	(junction
+		(at 45.72 46.99)
+		(diameter 0)
+		(color 0 0 0 0)
+	)
+	(junction
 		(at 177.8 116.84)
 		(diameter 0)
@@
 	(wire
 		(pts
+			(xy 45.72 46.99) (xy 45.72 49.53)
+		)
+		(stroke
+			(width 0)
+			(type default)
+		)
+	)
+	(wire
+		(pts
 			(xy 115.57 116.84) (xy 115.57 111.76)
 		)
@@
 	(wire
 		(pts
-			(xy 45.72 44.45) (xy 45.72 49.53)
+			(xy 45.72 44.45) (xy 45.72 46.99)
 		)
 		(stroke
@@
 	(wire
 		(pts
-			(xy 45.72 35.56) (xy 45.72 41.91)
+			(xy 45.72 35.56) (xy 45.72 39.37)
 		)
 		(stroke
@@
 	(wire
 		(pts
+			(xy 49.53 46.99) (xy 45.72 46.99)
+		)
+		(stroke
+			(width 0)
+			(type default)
+		)
+	)
+	(wire
+		(pts
 			(xy 187.96 116.84) (xy 177.8 116.84)
 		)
@@
 		(pts
 			(xy 166.37 133.35) (xy 166.37 138.43)
+		)
+		(stroke
+			(width 0)
+			(type default)
+		)
+	)
+	(wire
+		(pts
+			(xy 45.72 39.37) (xy 45.72 41.91)
+		)
+		(stroke
+			(width 0)
+			(type default)
+		)
+	)
+	(wire
+		(pts
+			(xy 45.72 39.37) (xy 49.53 39.37)
 		)
 		(stroke
@@
 			)
 		)
-		(property "Footprint" "Package_DIP:DIP-8_W7.62mm_Socket_LongPads"
+		(property "Footprint" "Package_SO:SOIC-8-1EP_3.9x4.9mm_P1.27mm_EP2.29x3mm"
 			(at 156.21 104.14 0)
 			(effects
@@
 			)
 		)
-		(property "Footprint" ""
+		(property "Footprint" "Capacitor_THT:C_Radial_D8.0mm_H11.5mm_P3.50mm"
 			(at 92.4052 69.85 0)
 			(effects
@@
 		(dnp no)
 		(fields_autoplaced yes)
-		(property "Reference" "PowerIn"
+		(property "Reference" "PowerIn1"
 			(at 34.925 36.83 0)
 			(effects
@@
 			(project "AmplifierCircuit"
 				(path "/1187d58b-5bff-4ac8-89f7-59cd1d310934/23e3ffa2-9d23-4864-a9b4-ed445dbced9e"
-					(reference "PowerIn")
+					(reference "PowerIn1")
 					(unit 1)
 				)
@@
 			)
 		)
-		(property "Footprint" ""
+		(property "Footprint" "Resistor_THT:R_Axial_DIN0309_L9.0mm_D3.2mm_P12.70mm_Horizontal"
 			(at 101.092 66.04 90)
 			(effects
@@
 			)
 		)
-		(property "Footprint" ""
+		(property "Footprint" "Resistor_THT:R_Axial_DIN0309_L9.0mm_D3.2mm_P12.70mm_Horizontal"
 			(at 113.792 66.04 90)
 			(effects
@@
 		(dnp no)
 		(fields_autoplaced yes)
-		(property "Reference" "RecieveCoil"
+		(property "Reference" "RecieveCoil1"
 			(at 103.505 111.76 0)
 			(effects
@@
 			)
 		)
-		(property "Footprint" ""
+		(property "Footprint" "Connector_PinSocket_2.54mm:PinSocket_1x02_P2.54mm_Vertical"
 			(at 102.87 119.38 0)
 			(effects
@@
 			(project "AmplifierCircuit"
 				(path "/1187d58b-5bff-4ac8-89f7-59cd1d310934/23e3ffa2-9d23-4864-a9b4-ed445dbced9e"
-					(reference "RecieveCoil")
+					(reference "RecieveCoil1")
 					(unit 1)
 				)
@@
 			)
 		)
-		(property "Footprint" ""
+		(property "Footprint" "Resistor_THT:R_Axial_DIN0309_L9.0mm_D3.2mm_P12.70mm_Horizontal"
 			(at 176.022 110.49 90)
 			(effects
@@
 			)
 		)
-		(property "Footprint" ""
+		(property "Footprint" "Capacitor_THT:C_Radial_D8.0mm_H11.5mm_P3.50mm"
 			(at 226.06 103.1748 0)
 			(effects
@@
 			)
 		)
-		(property "Footprint" ""
+		(property "Footprint" "Resistor_THT:R_Axial_DIN0309_L9.0mm_D3.2mm_P12.70mm_Horizontal"
 			(at 101.092 78.74 90)
 			(effects
@@
 	)
 	(symbol
+		(lib_id "Device:C")
+		(at 49.53 43.18 0)
+		(unit 1)
+		(exclude_from_sim no)
+		(in_bom yes)
+		(on_board yes)
+		(dnp no)
+		(fields_autoplaced yes)
+		(property "Reference" "C9"
+			(at 53.34 41.9099 0)
+			(effects
+				(font
+					(size 1.27 1.27)
+				)
+				(justify left)
+			)
+		)
+		(property "Value" "C"
+			(at 53.34 44.4499 0)
+			(effects
+				(font
+					(size 1.27 1.27)
+				)
+				(justify left)
+			)
+		)
+		(property "Footprint" "Capacitor_THT:C_Radial_D8.0mm_H11.5mm_P3.50mm"
+			(at 50.4952 46.99 0)
+			(effects
+				(font
+					(size 1.27 1.27)
+				)
+				(hide yes)
+			)
+		)
+		(property "Datasheet" "~"
+			(at 49.53 43.18 0)
+			(effects
+				(font
+					(size 1.27 1.27)
+				)
+				(hide yes)
+			)
+		)
+		(property "Description" "Unpolarized capacitor"
+			(at 49.53 43.18 0)
+			(effects
+				(font
+					(size 1.27 1.27)
+				)
+				(hide yes)
+			)
+		)
+		(pin "1"
+		)
+		(pin "2"
+		)
+		(instances
+			(project "AmplifierCircuit"
+				(path "/1187d58b-5bff-4ac8-89f7-59cd1d310934/23e3ffa2-9d23-4864-a9b4-ed445dbced9e"
+					(reference "C9")
+					(unit 1)
+				)
+			)
+		)
+	)
+	(symbol
 		(lib_id "Device:R")
 		(at 166.37 129.54 0)
@@
 			)
 		)
-		(property "Footprint" ""
+		(property "Footprint" "Resistor_THT:R_Axial_DIN0309_L9.0mm_D3.2mm_P12.70mm_Horizontal"
 			(at 164.592 129.54 90)
 			(effects
@@
 			)
 		)
-		(property "Footprint" ""
+		(property "Footprint" "Capacitor_THT:C_Radial_D8.0mm_H11.5mm_P3.50mm"
 			(at 167.3352 146.05 0)
 			(effects
@@
 		(dnp no)
 		(fields_autoplaced yes)
-		(property "Reference" "AudioOut"
+		(property "Reference" "AudioOut1"
 			(at 243.84 101.5999 0)
 			(effects
@@
 			(project "AmplifierCircuit"
 				(path "/1187d58b-5bff-4ac8-89f7-59cd1d310934/23e3ffa2-9d23-4864-a9b4-ed445dbced9e"
-					(reference "AudioOut")
+					(reference "AudioOut1")
 					(unit 1)
 				)
@@
 			)
 		)
-		(property "Footprint" "Package_DIP:DIP-8_W7.62mm_Socket_LongPads"
+		(property "Footprint" "Package_SO:SOIC-8-1EP_3.9x4.9mm_P1.27mm_EP2.29x3mm"
 			(at 62.23 43.18 0)
 			(effects
@@
 			)
 		)
-		(property "Footprint" ""
+		(property "Footprint" "Capacitor_THT:C_Radial_D8.0mm_H11.5mm_P3.50mm"
 			(at 116.5352 111.76 0)
 			(effects
@@
 			)
 		)
-		(property "Footprint" ""
+		(property "Footprint" "Capacitor_THT:C_Radial_D8.0mm_H11.5mm_P3.50mm"
 			(at 188.9252 114.3 0)
 			(effects
@@
 			)
 		)
-		(property "Footprint" ""
+		(property "Footprint" "Resistor_THT:R_Axial_DIN0309_L9.0mm_D3.2mm_P12.70mm_Horizontal"
 			(at 199.39 105.918 90)
 			(effects

Commit message: Updated the footprints for SMD
Parts:
- removed U2: ~, Package_SO:SOIC-8-1EP_3.9x4.9mm_P1.27mm_EP2.29x3mm, symbol HearingLoopLibrary:OPA209
- added U2: ~, Package_TO_SOT_SMD:SOT-23-5_HandSoldering, symbol HearingLoopLibrary:opa209
- renumbered RecieveCoil1 to LRx1, AudioOut1 to Out1, PowerIn1 to VinRx1
Connections:
- net GND2: now also U2.2 (V-)
- net VDD: now also U2.5 (V+)
- net at C7.2, R10.2, R9.1: now also U2.4 (-)
- net at C5.1, R8.2: now also U2.3 (+)
- net at C7.1, R10.1, R11.1: now also U2.1
